Commit message: MANY CHANGES, beginning development

File: baxter/baxter_description/urdf/baxter.urdf (robot description, URDF)
Before this commit: robot baxter, 49 links, 48 joints
Links:
- added link left_gripper_90, mass 0.0001
- added link left_realsense, mass 0.0001
- link left_gripper: geometry 
- link left_gripper_base: mass 0.0001 -> 0.3; geometry collision box size=0.12 0.15 0.05; collision cylinder length=0.068 radius=0.03
- link right_gripper: geometry 
- link right_gripper_base: mass 0.0001 -> 0.3; geometry collision cylinder length=0.08 radius=0.02; visual mesh filename=package://rethink_ee_description/meshes/pneumatic_gripper/p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
Joints:
- added joint left_endpoint_90: type fixed, parent left_gripper_base, child left_gripper_90, origin xyz=0.068 0 0.281597 rpy=0 1.57079632679 0
- added joint left_endpoint_realsense: type fixed, parent left_hand, child left_realsense, origin xyz=-0.1085 0 0.01 rpy=0 1.57 0
- joint head_pan: limit lower=-1.57079632679 upper=1.57079632679 effort=50000 velocity=10000 -> lower=-1.3963 upper=1.3963 effort=50000 velocity=10000
- joint left_endpoint: origin xyz=0.0 0 0.025 rpy=0 0 0 -> xyz=0 0 0.3745 rpy=0 0 0
- joint left_gripper_base: origin xyz=0 0 0 rpy=0 0 0 -> xyz=0 0 0.0 rpy=0 0 0
- joint left_s1: limit lower=-2.147 upper=1.047 effort=100.0 velocity=1.5 -> lower=-2.147 upper=1.047 effort=50.0 velocity=1.5
- joint right_endpoint: origin xyz=0.0 0 0.025 rpy=0 0 0 -> xyz=0 0 0.08 rpy=0 0 0
- joint right_gripper_base: origin xyz=0 0 0 rpy=0 0 0 -> xyz=0 0 0.0 rpy=0 0 0
- joint right_s1: limit lower=-2.147 upper=1.047 effort=100.0 velocity=1.5 -> lower=-2.147 upper=1.047 effort=50.0 velocity=1.5

File: baxter/baxter_description/urdf/baxter.urdf.xacro (robot description, xacro)
@@ -3,4 +3,6 @@
   <xacro:arg name="gazebo" default="false"/>
   <xacro:arg name="pedestal" default="true"/>
+  <xacro:arg name="left_arm" default="false"/>
+  <xacro:arg name="no_suction" default="false" />
   <!-- Baxter Base URDF -->
   <xacro:include filename="$(find baxter_description)/urdf/baxter_base/baxter_base.urdf.xacro">
@@ -13,7 +15,21 @@
     </xacro:include>
   </xacro:if>
-  <!-- Left End Effector -->
-  <xacro:include filename="$(find baxter_description)/urdf/left_end_effector.urdf.xacro" />
-  <!-- Right End Effector -->
-  <xacro:include filename="$(find baxter_description)/urdf/right_end_effector.urdf.xacro" />
+  <xacro:if value="$(arg no_suction)">
+      <xacro:include filename="$(find baxter_description)/urdf/apc_right_end_effector.urdf.xacro"/>
+      <xacro:include filename="$(find baxter_description)/urdf/apc_left_end_effector.urdf.xacro"/>
+  </xacro:if>
+  <xacro:unless value="$(arg no_suction)">
+      <xacro:if value="$(arg left_arm)">
+        <!-- Left End Effector -->
+        <xacro:include filename="$(find baxter_description)/urdf/left_end_effector.urdf.xacro"/>
+        <!-- Right End Effector -->
+        <xacro:include filename="$(find baxter_description)/urdf/apc_right_end_effector.urdf.xacro"/>
+      </xacro:if>
+      <xacro:unless value="$(arg left_arm)">
+        <!-- Right End Effector -->
+        <xacro:include filename="$(find baxter_description)/urdf/right_end_effector.urdf.xacro"/>
+        <!-- Left End Effector -->
+        <xacro:include filename="$(find baxter_description)/urdf/apc_left_end_effector.urdf.xacro"/>
+      </xacro:unless>
+  </xacro:unless>
 </robot>

File: baxter/baxter_description/urdf/baxter_base/baxter_base.urdf.xacro (robot description, xacro)
@@ -134,4 +134,11 @@
   </link>
   <link name="dummyhead1">
+    <!-- ADDED COLLISION MODEL FOR KINECT-->
+    <collision>
+        <origin rpy="0 0 0" xyz="0.0 0 0.25"/>
+        <geometry>
+          <cylinder length="0.1" radius="0.18"/>
+        </geometry>
+      </collision>
     <inertial>
       <origin rpy="0 0 0" xyz="0 0 0"/>
@@ -715,7 +722,26 @@
       </geometry>
     </collision>
+    <!-- NUC Collision Model -->
+    <!-- <collision>
+      <origin rpy="0 0 0" xyz="0.0 0.0 0.10"/>
+      <geometry>
+        <cylinder length="0.10" radius="0.07"/>
+      </geometry>
+    </collision> -->
+    <!-- NUC Visual -->
+    <!-- <visual>
+        <origin rpy="0 0 0" xyz="0.0 0.0 0.10"/>
+        <geometry>
+          <cylinder length="0.10" radius="0.07"/>
+        </geometry>
+        <material name="blue">
+          <color rgba="0 0 1 0.8"/>
+        </material>
+    </visual> -->
     <inertial>
       <origin rpy="0 0 0" xyz="0.02611 0.00159 -0.01117"/>
-      <mass value="2.07206"/>
+      <mass value = "3.07206"/>
+      <!--Added NUC mass value-->
+      <!--<mass value="2.07206"/>-->
       <inertia ixx="0.00711582686" ixy="0.00036036173" ixz="0.0007459496" iyy="0.01318227876" iyz="-0.00019663418" izz="0.00926852064"/>
     </inertial>

File: baxter/baxter_description/urdf/left_end_effector.urdf.xacro (robot description, xacro)
@@ -1,5 +1,5 @@
 <?xml version="1.0" ?>
 <robot name="left_end_effector" xmlns:xacro="http://www.ros.org/wiki/xacro">
-  <xacro:include filename="$(find rethink_ee_description)/urdf/pneumatic_gripper/rethink_pneumatic_gripper.xacro" />
-  <xacro:rethink_pneumatic_gripper side="left" />
+  <xacro:include filename="$(find apc_gripper_description)/urdf/apc_suction_gripper.xacro" />
+  <xacro:apc_suction_gripper side="left"/>
 </robot>

File: baxter/baxter_description/urdf/right_end_effector.urdf.xacro (robot description, xacro)
@@ -1,5 +1,5 @@
 <?xml version="1.0" ?>
 <robot name="right_end_effector" xmlns:xacro="http://www.ros.org/wiki/xacro">
-  <xacro:include filename="$(find rethink_ee_description)/urdf/pneumatic_gripper/rethink_pneumatic_gripper.xacro" />
-  <xacro:rethink_pneumatic_gripper side="right" />
+  <xacro:include filename="$(find apc_gripper_description)/urdf/apc_suction_gripper.xacro" />
+  <xacro:apc_suction_gripper side="right"/>
 </robot>
