Commit message: Many changes

File: baxter/apc_gripper_description/urdf/apc_suction_gripper.xacro (robot description, xacro)
@@ -16,10 +16,10 @@
     <!-- Base of end effector -->
     <link name="${side}_gripper_base">
-      <visual>
+      <!-- <visual>
         <origin rpy="0 -1.5708 0" xyz="0 0 0"/>
         <geometry>
           <mesh filename="package://apc_gripper_description/meshes/APC_Suction_Hand_2016.dae"/>
         </geometry>
-      </visual>
+      </visual> -->
       <collision>
       <!-- collision part for the realsense -->
@@ -30,4 +30,14 @@
         <material name="darkred">
           <color rgba=".5 .1 .1 1"/>
+        </material>
+      </collision>
+      <collision>
+      <!-- collision part for the realsense -->
+          <origin rpy="0 0 0" xyz="0.02 0 0.07"/>
+        <geometry>
+          <box size="0.09 0.1 0.06" />
+        </geometry>
+        <material name="darkred">
+          <color rgba=".1 .1 .5 1"/>
         </material>
       </collision>
@@ -61,5 +71,5 @@
     <!-- Distance from Realsense RGB Camera to centre of Baxter (left/right)_hand -->
     <joint name="${side}_endpoint_realsense" type="fixed">
-      <origin rpy="0.0 -1.85 0.0" xyz="-0.09 0.00 0.02"/>
+      <origin rpy="0.0698132 -1.97 0.0" xyz="-0.09 0.00 0.02"/>
       <parent link="${side}_hand"/>
       <child link="${side}_realsense"/>

File: baxter/baxter_description/urdf/baxter.urdf (robot description, URDF)
Before this commit: robot baxter, 51 links, 50 joints
Links:
- removed link left_gripper_90
- removed link left_realsense
- added link right_realsense, mass 0.0001
- link dummyhead1: geometry collision cylinder length=0.1 radius=0.18
- link left_gripper_base: geometry collision cylinder length=0.08 radius=0.02; visual mesh filename=package://rethink_ee_description/meshes/pneumatic_gripper/p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
- link left_lower_elbow: mass 2.07206 -> 3.07206
- link right_gripper_base: mass 0.3 -> 0.5; geometry collision box size=0.09 0.1 0.06; collision box size=0.1 0.15 0.03
Joints:
- removed joint left_endpoint_90
- removed joint left_endpoint_realsense
- added joint right_endpoint_realsense: type fixed, parent right_hand, child right_realsense, origin xyz=-0.09 0.00 0.02 rpy=0.0698132 -1.97 0.0
- joint left_endpoint: origin xyz=0 0 0.3745 rpy=0 0 0 -> xyz=0 0 0.08 rpy=0 0 0

File: baxter/baxter_description/urdf/baxter.urdf.xacro (robot description, xacro)
@@ -5,4 +5,6 @@
   <xacro:arg name="left_arm" default="false"/>
   <xacro:arg name="no_suction" default="false" />
+  <xacro:property name="pi" value="3.14159265359" />
+  <xacro:property name="tip_length" value="${0.06 + 0.02}" />
   <!-- Baxter Base URDF -->
   <xacro:include filename="$(find baxter_description)/urdf/baxter_base/baxter_base.urdf.xacro">

Commit message: Updated Baxter description with old gripper design

File: baxter/apc_gripper_description/urdf/apc_suction_gripper.xacro (robot description, xacro)
@@ -33,8 +33,8 @@
       </collision>
       <collision>
-      <!-- collision part for the realsense -->
-          <origin rpy="0 0 0" xyz="0.02 0 0.07"/>
+      <!-- collision part for the suction tubes -->
+          <origin rpy="0 0 0" xyz="0.02 0 0.055"/>
         <geometry>
-          <box size="0.09 0.1 0.06" />
+          <box size="0.04 0.07 0.03" />
         </geometry>
         <material name="darkred">

File: baxter/baxter_description/urdf/baxter.urdf (robot description, URDF)
Before this commit: robot baxter, 50 links, 49 joints
Links:
- link right_gripper_base: geometry collision box size=0.04 0.07 0.03; collision box size=0.1 0.15 0.03
